File: fw16_oculink8i.kicad_sch (KiCad schematic)
At the start: 35 parts, among them J1 FXBeam, J2 Fan0, J3 Fan1, J4 173162-0131, U1 BR24G32FVT-3GE2

Commit message: working rev1.1
Parts:
- removed R15, R22: 0R, Resistor_SMD:R_0402_1005Metric, symbol Device:R
- R14: now fitted
- R23: now not fitted
Changed lines of the file:
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@@
 	)
 	(junction
-		(at 113.03 199.39)
-		(diameter 0)
-		(color 0 0 0 0)
-	)
-	(junction
 		(at 36.83 199.39)
 		(diameter 0)
@@
 	(wire
 		(pts
-			(xy 113.03 199.39) (xy 120.65 199.39)
-		)
-		(stroke
-			(width 0)
-			(type default)
-		)
-	)
-	(wire
-		(pts
 			(xy 260.35 176.53) (xy 278.13 176.53)
 		)
@@
 	(wire
 		(pts
-			(xy 104.14 199.39) (xy 113.03 199.39)
-		)
-		(stroke
-			(width 0)
-			(type default)
-		)
-	)
-	(wire
-		(pts
 			(xy 73.66 113.03) (xy 83.82 113.03)
 		)
@@
 	(wire
 		(pts
-			(xy 106.68 205.74) (xy 104.14 205.74)
-		)
-		(stroke
-			(width 0)
-			(type default)
-		)
-	)
-	(wire
-		(pts
 			(xy 219.71 144.78) (xy 220.98 143.51)
 		)
@@
 	(wire
 		(pts
-			(xy 106.68 205.74) (xy 113.03 199.39)
-		)
-		(stroke
-			(width 0)
-			(type default)
-		)
-	)
-	(wire
-		(pts
 			(xy 100.33 83.82) (xy 109.22 83.82)
 		)
@@
 	(wire
 		(pts
-			(xy 93.98 193.04) (xy 96.52 193.04)
-		)
-		(stroke
-			(width 0)
-			(type default)
-		)
-	)
-	(wire
-		(pts
 			(xy 360.68 107.95) (xy 358.14 107.95)
 		)
@@
 	(wire
 		(pts
-			(xy 73.66 201.93) (xy 90.17 201.93)
+			(xy 73.66 201.93) (xy 88.9 201.93)
 		)
 		(stroke
@@
 	(wire
 		(pts
-			(xy 106.68 193.04) (xy 104.14 193.04)
+			(xy 100.33 196.85) (xy 110.49 196.85)
 		)
 		(stroke
@@
 	(wire
 		(pts
-			(xy 93.98 205.74) (xy 96.52 205.74)
-		)
-		(stroke
-			(width 0)
-			(type default)
-		)
-	)
-	(wire
-		(pts
 			(xy 255.27 184.15) (xy 255.27 186.69)
 		)
@@
 	(wire
 		(pts
-			(xy 106.68 193.04) (xy 113.03 199.39)
-		)
-		(stroke
-			(width 0)
-			(type default)
-		)
-	)
-	(wire
-		(pts
 			(xy 360.68 130.81) (xy 358.14 130.81)
 		)
@@
 	(wire
 		(pts
-			(xy 360.68 138.43) (xy 358.14 138.43)
+			(xy 73.66 199.39) (xy 88.9 199.39)
 		)
 		(stroke
@@
 	(wire
 		(pts
-			(xy 358.14 105.41) (xy 373.38 105.41)
+			(xy 360.68 138.43) (xy 358.14 138.43)
 		)
 		(stroke
@@
 	(wire
 		(pts
-			(xy 358.14 59.69) (xy 373.38 59.69)
+			(xy 358.14 105.41) (xy 373.38 105.41)
 		)
 		(stroke
@@
 	(wire
 		(pts
-			(xy 358.14 57.15) (xy 373.38 57.15)
+			(xy 358.14 59.69) (xy 373.38 59.69)
 		)
 		(stroke
@@
 	(wire
 		(pts
-			(xy 73.66 199.39) (xy 96.52 199.39)
+			(xy 358.14 57.15) (xy 373.38 57.15)
 		)
 		(stroke
@@
 	(wire
 		(pts
-			(xy 93.98 205.74) (xy 90.17 201.93)
-		)
-		(stroke
-			(width 0)
-			(type default)
-		)
-	)
-	(wire
-		(pts
 			(xy 264.16 40.64) (xy 247.65 40.64)
 		)
@@
 	(wire
 		(pts
-			(xy 90.17 196.85) (xy 93.98 193.04)
-		)
-		(stroke
-			(width 0)
-			(type default)
-		)
-	)
-	(wire
-		(pts
 			(xy 36.83 201.93) (xy 36.83 199.39)
 		)
@@
 	(wire
 		(pts
-			(xy 73.66 196.85) (xy 90.17 196.85)
+			(xy 73.66 196.85) (xy 92.71 196.85)
 		)
 		(stroke
@@
 	)
 	(label "PERSTA"
-		(at 120.65 199.39 180)
+		(at 110.49 196.85 180)
 		(effects
 			(font
@@
 	(symbol
 		(lib_id "Device:R")
-		(at 100.33 193.04 90)
+		(at 96.52 196.85 90)
 		(unit 1)
 		(exclude_from_sim no)
 		(in_bom yes)
 		(on_board yes)
-		(dnp yes)
+		(dnp no)
 		(property "Reference" "R14"
-			(at 100.33 191.008 90)
+			(at 96.52 194.818 90)
 			(effects
 				(font
@@
 		)
 		(property "Value" "0R"
-			(at 100.33 195.072 90)
+			(at 96.52 198.882 90)
 			(effects
 				(font
@@
 		)
 		(property "Footprint" "Resistor_SMD:R_0402_1005Metric"
-			(at 100.33 194.818 90)
+			(at 96.52 198.628 90)
 			(effects
 				(font
@@
 		)
 		(property "Datasheet" "~"
-			(at 100.33 193.04 0)
+			(at 96.52 196.85 0)
 			(effects
 				(font
@@
 		)
 		(property "Description" "Resistor"
-			(at 100.33 193.04 0)
+			(at 96.52 196.85 0)
 			(effects
 				(font
@@
 	)
 	(symbol
-		(lib_id "Device:R")
-		(at 100.33 199.39 90)
-		(unit 1)
-		(exclude_from_sim no)
-		(in_bom yes)
-		(on_board yes)
-		(dnp yes)
-		(property "Reference" "R15"
-			(at 100.33 197.358 90)
-			(effects
-				(font
-					(size 1.27 1.27)
-				)
-			)
-		)
-		(property "Value" "0R"
-			(at 100.33 201.422 90)
-			(effects
-				(font
-					(size 1.27 1.27)
-				)
-			)
-		)
-		(property "Footprint" "Resistor_SMD:R_0402_1005Metric"
-			(at 100.33 201.168 90)
-			(effects
-				(font
-					(size 1.27 1.27)
-				)
-				(hide yes)
-			)
-		)
-		(property "Datasheet" "~"
-			(at 100.33 199.39 0)
-			(effects
-				(font
-					(size 1.27 1.27)
-				)
-				(hide yes)
-			)
-		)
-		(property "Description" "Resistor"
-			(at 100.33 199.39 0)
-			(effects
-				(font
-					(size 1.27 1.27)
-				)
-				(hide yes)
-			)
-		)
-		(pin "2"
-		)
-		(pin "1"
-		)
-		(instances
-			(project "fw16_oculink8i"
-				(path "/50f5fd03-67f8-43d1-8bfe-dca2cf908bf0"
-					(reference "R15")
-					(unit 1)
-				)
-			)
-		)
-	)
-	(symbol
 		(lib_id "Device:R_Small")
 		(at 234.95 110.49 0)
@@
 		(in_bom yes)
 		(on_board yes)
-		(dnp no)
+		(dnp yes)
 		(property "Reference" "R23"
 			(at 96.52 81.788 90)
@@
 					(unit 1)
 				)
-			)
-		)
-	)
-	(symbol
-		(lib_id "Device:R")
-		(at 100.33 205.74 90)
-		(unit 1)
-		(exclude_from_sim no)
-		(in_bom yes)
-		(on_board yes)
-		(dnp yes)
-		(property "Reference" "R22"
-			(at 100.33 203.708 90)
-			(effects
-				(font
-					(size 1.27 1.27)
-				)
-			)
-		)
-		(property "Value" "0R"
-			(at 100.33 207.772 90)
-			(effects
-				(font
-					(size 1.27 1.27)
-				)
-			)
-		)
-		(property "Footprint" "Resistor_SMD:R_0402_1005Metric"
-			(at 100.33 207.518 90)
-			(effects
-				(font
-					(size 1.27 1.27)
-				)
-				(hide yes)
-			)
-		)
-		(property "Datasheet" "~"
-			(at 100.33 205.74 0)
-			(effects
-				(font
-					(size 1.27 1.27)
-				)
-				(hide yes)
-			)
-		)
-		(property "Description" "Resistor"
-			(at 100.33 205.74 0)
-			(effects
-				(font
-					(size 1.27 1.27)
-				)
-				(hide yes)
-			)
-		)
-		(pin "2"
-		)
-		(pin "1"
-		)
-		(instances
-			(project "fw16_oculink8i"
-				(path "/50f5fd03-67f8-43d1-8bfe-dca2cf908bf0"
-					(reference "R22")
-					(unit 1)
-				)
