File: fw16_oculink8i.kicad_sch (KiCad schematic)
At the start: 33 parts, among them J1 FXBeam, J2 Fan0, J3 Fan1, J4 173162-0131, U1 BR24G32FVT-3GE2

Commit message: finalized rev1.2 order
Parts:
- removed J1: FXBeam, Expansion_Bay:FXBeam, symbol Expansion_Bay:FXBeam
- removed J4: 173162-0131, Nano_Pitch:Nano-Pitch-173162-0131_JLC-DRC, symbol Nano_Pitch:173162-0131
- removed R1: 330K, Resistor_SMD:R_0402_1005Metric, symbol Device:R
- removed R12: R, Resistor_SMD:R_0402_1005Metric, symbol Device:R_Small
- removed R13: 1K, Resistor_SMD:R_0402_1005Metric, symbol Device:R_Small
- removed R14, R23: 0R, Resistor_SMD:R_0402_1005Metric, symbol Device:R
- removed TP1, TP2: TestPoint, TestPoint:TestPoint_Pad_D1.0mm, symbol Connector:TestPoint
- added C1, C2, C4, C5: 0.1U, Capacitor_SMD:C_0402_1005Metric, symbol Device:C_Small
- added J3: FXBeam, Expansion_Bay:FXBeam, symbol Expansion_Bay:FXBeam_MultiUnit
- added J4: I2C, Connector_JST:JST_SH_SM04B-SRSS-TB_1x04-1MP_P1.00mm_Horizontal, symbol Connector_Generic_MountingPin:Conn_01x04_MountingPin
- added J5: USB_A, USB:87583-2010BLF, symbol Connector:USB_A
- added J6: x8 NPIO, Nano_Pitch:Nano-Pitch-173162-0132, symbol Nano_Pitch:Nano_Pitch-173162
- added R16: 1K, Resistor_SMD:R_0402_1005Metric, symbol Device:R_Small
- added R2: 330K, Resistor_SMD:R_0402_1005Metric, symbol Device:R
- added R20: 10K, Resistor_SMD:R_0402_1005Metric, symbol Device:R_Small
- added R22, R23, R28, R3, R30, R31, R33, R34, R4: 0R, Resistor_SMD:R_0402_1005Metric, symbol Device:R_Small
- added R24, R25: 9K1, Resistor_SMD:R_0402_1005Metric, symbol Device:R_Small
- added R26, R27: 3K9, Resistor_SMD:R_0402_1005Metric, symbol Device:R_Small
- added R29, R32: 100K, Resistor_SMD:R_0402_1005Metric, symbol Device:R_Small
- added R35: 0R, Resistor_SMD:R_0402_1005Metric, symbol Device:R
- added SW1: SW_DPDT_x2, Switches:SSSS820101, symbol Switch:SW_DPDT_x2
- added SW2: SW_DIP_x02, Button_Switch_SMD:SW_DIP_SPSTx02_Slide_Copal_CHS-02B_W7.62mm_P1.27mm, symbol Switch:SW_DIP_x02
- added TP1, TP2, TP3: TestPoint_Small, TestPoint:TestPoint_Pad_D1.0mm, symbol Connector:TestPoint_Small
- added U2, U3: TL331LV, Package_TO_SOT_SMD:SOT-23-5, symbol Comparator:TL331
- H1, H2, H3, H4: footprint Expansion_Bay:MountingHole_6.2mm -> Expansion_Bay:MountingHole_6.2mm_EasySolder_Cut
- J1: renamed from J2; value Fan0 -> Fan; footprint fpc-fan:JUSHUO_AFC05-S04FIA-00 -> FPC_Conn:AFC58-S04FIA_4Pin; Part Nr. JUSHUO AFC05-S04FIA-00 -> AFC58-S04FIA; now left out of the parts list
- J2: renamed from J3; value Fan1 -> Fan; footprint fpc-fan:JUSHUO_AFC05-S04FIA-00 -> FPC_Conn:AFC58-S04FIA_4Pin; Part Nr. JUSHUO AFC05-S04FIA-00 -> AFC58-S04FIA; now left out of the parts list
- R17, R21: value 0R -> 1K
- R18: value 0R -> 10K; now not fitted
- R19: value 100K -> 1K
- renumbered C1 to C3, R2 to R1, R20 to R10, R3 to R11, R8 to R12, R9 to R13, R6 to R14, R7 to R15, R16 to R5, R5 to R6, R10 to R7, R11 to R8, R4 to R9
Connections:
- net 12V_FAN: now also C1.2, C2.2, J3.PL4 (12V_FAN)
- net 3V3_EEPROM: now also J4.2 (Pin_2)
- net CPRSNTA: now also J6.B12, R28.1; no longer R19.1
- net CPRSNTB: now also J6.B33, R31.1
- net FAN0_PWM: now also J3.PL5 (Fan0_PWM)
- net FAN0_SPD: now also J3.PH2 (Fan0_SPEED)
- net FAN1_PWM: now also J3.PK5 (Fan1_PWM)
- net FAN1_SPD: now also J3.PJ2 (Fan1_SPEED)
- net GND: now also R17.1, C1.1, C2.1, C4.2, C5.2, J3.PA3 (GND), J3.PA6 (GND), J3.PB3 (GND), J3.PB6 (GND), J3.PC6 (GND), J3.PD1 (GND), J3.PD2 (GND), J3.PD6 (GND), J3.PE1 (GND), J3.PE2 (GND), J3.PE3 (GND), J3.PE6 (GND), J3.PF1 (GND), J3.PF6 (GND), J3.PG6 (GND), J3.PH3 (GND), J3.PH6 (GND), J3.PH7 (GND), J3.PH8 (GND), J3.PJ6 (GND), J3.PJ7 (GND), J3.PJ8 (GND), J3.PK4 (GND), J3.PK6 (GND), J3.PL3 (GND), J3.PL6 (GND), J3.SB2 (GND), J3.SB7 (GND), J3.SC1 (GND), J3.SC3 (GND), J3.SC6 (GND), J3.SC8 (GND), J3.SE2 (GND), J3.SE7 (GND), J3.SF1 (GND), J3.SF3 (GND), J3.SF6 (GND), J3.SF8 (GND), J3.SH2 (GND), J3.SH7 (GND), J3.SJ1 (GND), J3.SJ3 (GND), J3.SJ6 (GND), J3.SJ8 (GND), J4.1 (Pin_1), J4.MP (MountPin), J5.4 (GND), J6.A1, J6.A10, J6.A13, J6.A16, J6.A19, J6.A22, J6.A25, J6.A28, J6.A31, J6.A34, J6.A37, J6.A4, J6.A40, J6.A7, J6.B1, J6.B10, J6.B13, J6.B16, J6.B19, J6.B22, J6.B25, J6.B28, J6.B31, J6.B34, J6.B37, J6.B4, J6.B40, J6.B7, R16.1, R2.1, R26.1, R27.1, R34.2, R35.2, U2.2 (V-), U3.2 (V-)
- net I2C_SCL: now also J3.PC3 (I2C_CLK_ALW), R4.2; no longer R17.2
- net I2C_SDA: now also J3.PD3 (I2C_DAT_ALW), R3.1; no longer R18.2
- net PERSTA: now also J6.B11, SW1.2 (B)
- net PERSTB: now also J6.B32, SW1.5 (B)
- net REFCLKA+: now also J3.SC2 (PEX_REFCLK), J6.A12
- net REFCLKA-: now also J3.SD2 (PEX_REFCLK#), J6.A11
- net REFCLKB+: now also J3.SK7 (DP_A_AUXP), J6.A32
- net REFCLKB-: now also J3.SJ7 (DP_A_AUXN), J6.A33
- net RX0+: now also J3.SE8 (PEX_RX0P), J6.A3
- net RX0-: now also J3.SD8 (PEX_RX0N), J6.A2
- net RX1+: now also J3.SB8 (PEX_RX1P), J6.A5
- net RX1-: now also J3.SA8 (PEX_RX1N), J6.A6
- net RX2+: now also J3.SE6 (PEX_RX2P), J6.A14
- net RX2-: now also J3.SD6 (PEX_RX2N), J6.A15
- net RX3+: now also J3.SB6 (PEX_RX3P), J6.A18
- net RX3-: now also J3.SA6 (PEX_RX3N), J6.A17
- net RX4+: now also J3.SA3 (PEX_RX4P), J6.A24
- net RX4-: now also J3.SB3 (PEX_RX4N), J6.A23
- net RX5+: now also J3.SD3 (PEX_RX5P), J6.A26
- net RX5-: now also J3.SE3 (PEX_RX5N), J6.A27
- net RX6+: now also J3.SA1 (PEX_RX6P), J6.A36
- net RX6-: now also J3.SB1 (PEX_RX6N), J6.A35
- net RX7+: now also J3.SE1 (PEX_RX7P), J6.A39
- net RX7-: now also J3.SD1 (PEX_RX7N), J6.A38
- net SSD1_RST: now also J3.PF3 (SSD1_RST#), SW1.1 (A)
- net SSD2_RST: now also J3.PG3 (SSD2_RST#), SW1.4 (A)
- net TX0+: now also J3.SH8 (PEX_TX0P), J6.B3
- net TX0-: now also J3.SG8 (PEX_TX0N), J6.B2
- net TX1+: now also J3.SL8 (PEX_TX1P), J6.B6
- net TX1-: now also J3.SK8 (PEX_TX1N), J6.B5
- net TX2+: now also J3.SG6 (PEX_TX2P), J6.B14
- net TX2-: now also J3.SH6 (PEX_TX2N), J6.B15
- net TX3+: now also J3.SL6 (PEX_TX3P), J6.B18
- net TX3-: now also J3.SK6 (PEX_TX3N), J6.B17
- net TX4+: now also J3.SK3 (PEX_TX4P), J6.B24
- net TX4-: now also J3.SL3 (PEX_TX4N), J6.B23
- net TX5+: now also J3.SH3 (PEX_TX5P), J6.B26
- net TX5-: now also J3.SG3 (PEX_TX5N), J6.B27
- net TX6+: now also J3.SK1 (PEX_TX6P), J6.B36
- net TX6-: now also J3.SL1 (PEX_TX6N), J6.B35
- net TX7+: now also J3.SH1 (PEX_TX7P), J6.B38
- net TX7-: now also J3.SG1 (PEX_TX7N), J6.B39
- net CLK_AUTO_EN2: now reaches R21.1
- net CLK_AUTO_EN2: now also U3.4
- net at R1.2: now also J3.SL2 (ID1)
- net at R6.1, U1.5 (SDA): now also J4.3 (Pin_3), R3.2; no longer R18.1
- net at R9.2, U1.6 (SCL): now also J4.4 (Pin_4), R4.1; no longer R17.1
- net 3V3_ALW renamed 3V3_ID
- net 3V3_ID: now also J3.PA5 (3V3_ALW), J3.PB5 (3V3_ALW); no longer R19.2
- net CLKREQ renamed CLKREQ2
- net CLKREQ2: now also J3.PG2 (SSD2_CLK_REQ#), R20.2, SW2.3
- new net: J6.MP (Shield), R35.1
- new net: R24.2, R26.2, U2.1 (-)
- new net: R28.2, R29.1, U2.3 (+)
- new net: R16.2, SW2.1
- new net: R17.2, SW2.2
- new net: R29.2, R30.2
- new net: R25.2, R27.2, U3.1 (-)
- new net: R31.2, R32.1, U3.3 (+)
- new net: J5.5 (Shield), R34.1
- new net: R32.2, R33.2
- new net: J3.PJ1 (ID0), R2.2
- new net 3V3_CLK_EN1: C4.1, R22.1, R24.1, U2.5 (V+)
- new net 3V3_CLK_EN2: C5.1, R23.2, R25.1, U3.5 (V+)
- new net 3V3_CTRL: J3.PA4 (3V3_ALW), J3.PB4 (3V3_ALW), R18.1, R20.1, R22.2, R23.1, R30.1, R33.1
- new net 5V_ALW: J3.PK7 (5V_ALW), J3.PK8 (5V_ALW), J3.PL7 (5V_ALW), J3.PL8 (5V_ALW), J5.1 (VBUS)
- new net CLKREQ1: J3.SA4 (PEX_CLK_REQ#), R18.2, R19.2, SW2.4
- new net CLK_AUTO_EN1: R19.1, U2.4
- new net GPIO0: J3.PG1 (GPIO0_EC), TP3.1
- new net GPIO1: J3.PH1 (GPIO1_EC), TP2.1
- new net PEX_RST: J3.SA5 (PEX_RST#), SW1.3 (C), SW1.6 (C)
- new net PWR_GOOD: J3.PL1 (PWR_GOOD), TP1.1
- new net USB+: J3.PJ3 (USB+), J5.3 (D+)
- new net USB-: J3.PK3 (USB-), J5.2 (D-)
Other:
- note added: "Pull-down on device side"
- note added: "Pull-up to 3.3V"
- note removed: "TODO: Add CPRSNT logic"
- title: (none) -> FXBeam to OCuLink Adapter
- moved on the sheet: C3, H1, H2, H3, H4, J1, J2, R1, R10, R11, R12, R13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

Commit message: finalize rev1.3
Parts:
- added R36: 0R, Resistor_SMD:R_0402_1005Metric, symbol Device:R_Small
- J5: now not fitted
- R24, R25: value 9K1 -> 100K
- R26, R27: value 3K9 -> 47K
- R28, R31: value 0R -> 1K
Connections:
- net PEX_RST: now also R36.2; no longer SW1.6 (C)
- new net: R36.1, SW1.6 (C)
Other:
- note added: "Floating by default"
Changed lines of the file:
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@@
 		)
 	)
+	(text "Floating by default"
+		(exclude_from_sim no)
+		(at 357.632 47.752 0)
+		(effects
+			(font
+				(size 1.27 1.27)
+			)
+		)
+	)
 	(text "Pull-down on device side"
 		(exclude_from_sim no)
@@
 	(wire
 		(pts
+			(xy 369.57 50.8) (xy 370.84 50.8)
+		)
+		(stroke
+			(width 0)
+			(type default)
+		)
+	)
+	(wire
+		(pts
 			(xy 365.76 85.09) (xy 364.49 83.82)
 		)
@@
 	(wire
 		(pts
-			(xy 360.68 50.8) (xy 370.84 50.8)
+			(xy 354.33 50.8) (xy 364.49 50.8)
 		)
 		(stroke
@@
 	)
 	(label "PEX_RST"
-		(at 360.68 50.8 0)
+		(at 354.33 50.8 0)
 		(effects
 			(font
@@
 			)
 		)
-		(property "Value" "3K9"
+		(property "Value" "47K"
 			(at 314.198 57.15 90)
 			(effects
@@
 	(symbol
 		(lib_id "Device:R_Small")
+		(at 367.03 50.8 270)
+		(mirror x)
+		(unit 1)
+		(exclude_from_sim no)
+		(in_bom yes)
+		(on_board yes)
+		(dnp yes)
+		(property "Reference" "R36"
+			(at 367.03 52.324 90)
+			(effects
+				(font
+					(size 1.016 1.016)
+				)
+			)
+		)
+		(property "Value" "0R"
+			(at 367.03 49.022 90)
+			(effects
+				(font
+					(size 1.016 1.016)
+				)
+			)
+		)
+		(property "Footprint" "Resistor_SMD:R_0402_1005Metric"
+			(at 367.03 50.8 0)
+			(effects
+				(font
+					(size 1.27 1.27)
+				)
+				(hide yes)
+			)
+		)
+		(property "Datasheet" "~"
+			(at 367.03 50.8 0)
+			(effects
+				(font
+					(size 1.27 1.27)
+				)
+				(hide yes)
+			)
+		)
+		(property "Description" "Resistor, small symbol"
+			(at 367.03 50.8 0)
+			(effects
+				(font
+					(size 1.27 1.27)
+				)
+				(hide yes)
+			)
+		)
+		(pin "2"
+		)
+		(pin "1"
+		)
+		(instances
+			(project "fw16_oculink8i"
+				(path "/50f5fd03-67f8-43d1-8bfe-dca2cf908bf0"
+					(reference "R36")
+					(unit 1)
+				)
+			)
+		)
+	)
+	(symbol
+		(lib_id "Device:R_Small")
 		(at 379.73 95.25 90)
 		(mirror x)
@@
 			)
 		)
-		(property "Value" "3K9"
+		(property "Value" "47K"
 			(at 314.198 96.52 90)
 			(effects
@@
 			)
 		)
-		(property "Value" "9K1"
+		(property "Value" "100K"
 			(at 307.34 94.488 90)
 			(effects
@@
 			)
 		)
-		(property "Value" "0R"
+		(property "Value" "1K"
 			(at 281.94 89.408 90)
 			(effects
@@
 		(in_bom yes)
 		(on_board yes)
-		(dnp no)
+		(dnp yes)
 		(fields_autoplaced yes)
 		(property "Reference" "J5"
@@
 			)
 		)
-		(property "Value" "9K1"
+		(property "Value" "100K"
 			(at 307.34 55.118 90)
 			(effects
@@
 			)
 		)
-		(property "Value" "0R"
+		(property "Value" "1K"
 			(at 281.94 50.038 90)
 			(effects
