File: fw16_oculink8i.kicad_sch (KiCad schematic)
At the start: 59 parts, among them J1 Fan, J2 Fan, J3 FXBeam, J4 I2C, J5 USB_A, J6 x8 NPIO, SW1 SW_DPDT_x2, SW2 SW_DIP_x02, U1 BR24G32FVT-3GE2, U2 TL331LV, U3 TL331LV

Commit message: finalize rev1.3 for real now... maybe
Parts:
- removed R35: 0R, Resistor_SMD:R_0402_1005Metric, symbol Device:R
- removed TP1, TP2, TP3: TestPoint_Small, TestPoint:TestPoint_Pad_D1.0mm, symbol Connector:TestPoint_Small
Connections:
- net GND: now also J6.MP (Shield)
- net REFCLKA+: now also J6.A11; no longer J6.A12
- net REFCLKA-: now also J6.A12; no longer J6.A11
- net REFCLKB+: now also J6.A33; no longer J6.A32
- net REFCLKB-: now also J6.A32; no longer J6.A33
- net RX6+: now also J6.A35; no longer J6.A36
- net RX6-: now also J6.A36; no longer J6.A35
- net RX7+: now also J6.A38; no longer J6.A39
- net RX7-: now also J6.A39; no longer J6.A38
- net PWR_GOOD: no longer names the net of J3.PL1 (PWR_GOOD)
