File: fw16_oculink8i.kicad_pcb (KiCad board)
At the start: 4 copper layers, 118.7 x 72.5 mm, 35 parts, among them J1 FXBeam, J2 Fan0, J3 Fan1, J4 173162-0131, U1 BR24G32FVT-3GE2

Commit message: working rev1.1
Parts:
- removed R15, R22: 0R, Resistor_SMD:R_0402_1005Metric
Routing:
- net /SSD2_RST: track 19.9 -> 0.00 mm
- net /SSD2_CLKREQ: track 17.3 -> 0.00 mm
- net /PERSTA: track 83.6 -> 79.7 mm
- net /SSD1_RST: track 20.1 -> 16.7 mm

Commit message: finalized rev1.2 order
Parts:
- removed the R12 at (95.4, 84.3)
- removed the R13 at (95.4, 83.2)
- removed the R14 at (95.4, 78.5)
- added C1: 0.1U, Capacitor_SMD:C_0402_1005Metric, F.Cu at (140.8, 93.3)
- added C2: 0.1U, Capacitor_SMD:C_0402_1005Metric, F.Cu at (61.9, 88.7)
- added C4: 0.1U, Capacitor_SMD:C_0402_1005Metric, F.Cu at (84.2, 61.4)
- added C5: 0.1U, Capacitor_SMD:C_0402_1005Metric, F.Cu at (92.7, 61.4)
- added J5: USB_A, USB:87583-2010BLF, F.Cu at (57.8, 42.5)
- added J6: x8 NPIO, Nano_Pitch:Nano-Pitch-173162-0132, F.Cu at (131.8, 28.6)
- added R10: 0R, Resistor_SMD:R_0402_1005Metric, F.Cu at (83.3, 75.8)
- added R11: 100K, Resistor_SMD:R_0402_1005Metric, F.Cu at (85.4, 75.8)
- added R16: 1K, Resistor_SMD:R_0402_1005Metric, F.Cu at (84.4, 70.3)
- added R22: 0R, Resistor_SMD:R_0402_1005Metric, F.Cu at (84.2, 60.3)
- added R24: 9K1, Resistor_SMD:R_0402_1005Metric, F.Cu at (84.2, 58.8)
- added R25: 9K1, Resistor_SMD:R_0402_1005Metric, F.Cu at (92.7, 58.8)
- added R26: 3K9, Resistor_SMD:R_0402_1005Metric, F.Cu at (84.2, 57.7)
- added R27: 3K9, Resistor_SMD:R_0402_1005Metric, F.Cu at (92.7, 57.7)
- added R28: 0R, Resistor_SMD:R_0402_1005Metric, F.Cu at (80.1, 56.0)
- added R29: 47K, Resistor_SMD:R_0402_1005Metric, F.Cu at (81.2, 56.0)
- added R3: 0R, Resistor_SMD:R_0402_1005Metric, F.Cu at (86.1, 81.0)
- added R30: 0R, Resistor_SMD:R_0402_1005Metric, F.Cu at (82.3, 56.0)
- added R31: 0R, Resistor_SMD:R_0402_1005Metric, F.Cu at (88.7, 56.0)
- added R32: 47K, Resistor_SMD:R_0402_1005Metric, F.Cu at (89.7, 56.0)
- added R33: 0R, Resistor_SMD:R_0402_1005Metric, F.Cu at (90.9, 56.0)
- added R34: 0R, Resistor_SMD:R_0402_1005Metric, F.Cu at (47.1, 42.1)
- added R4: 0R, Resistor_SMD:R_0402_1005Metric, F.Cu at (86.8, 80.3)
- added SW1: SW_DPDT_x2, Switches:SSSS820101, F.Cu at (78.0, 67.4)
- added SW2: SW_DIP_x02, Button_Switch_SMD:SW_DIP_SPSTx02_Slide_Copal_CHS-02B_W7.62mm_P1.27mm, F.Cu at (88.3, 66.4)
- added TP3: TestPoint_Small, TestPoint:TestPoint_Pad_D1.0mm, F.Cu at (91.5, 73.4)
- added U2: TL331LV, Package_TO_SOT_SMD:SOT-23-5, F.Cu at (81.2, 59.2)
- added U3: TL331LV, Package_TO_SOT_SMD:SOT-23-5, F.Cu at (89.8, 59.2)
- H1, H2, H3, H4: footprint Expansion_Bay:MountingHole_6.2mm -> Expansion_Bay:MountingHole_6.2mm_EasySolder_Cut
- J1: renamed from J2; value Fan0 -> Fan; footprint fpc-fan:JUSHUO_AFC05-S04FIA-00 -> FPC_Conn:AFC58-S04FIA_4Pin
- J2: renamed from J3; value Fan1 -> Fan; footprint fpc-fan:JUSHUO_AFC05-S04FIA-00 -> FPC_Conn:AFC58-S04FIA_4Pin
- J4: value 173162-0131 -> I2C; footprint Nano_Pitch:Nano-Pitch-173162-0131_JLC-DRC -> Connector_JST:JST_SH_SM04B-SRSS-TB_1x04-1MP_P1.00mm_Horizontal
- R17, R21: value 0R -> 1K
- R18, R20: value 0R -> 10K
- R19: value 100K -> 1K
- R5: renamed from R3; value 100K -> 0R
- TP1, TP2: value TestPoint -> TestPoint_Small
- moved J4 78.9 mm to (72.1, 82.1), turned to 90 degrees
- moved R35 59.8 mm to (118.2, 29.9), turned to -90 degrees
- moved R1 48.4 mm to (84.0, 84.9), turned to 0 degrees
- moved R18 24.2 mm to (80.4, 62.4), turned to -90 degrees
- moved R21 22.6 mm to (90.0, 62.4), turned to -90 degrees
- moved R19 21.7 mm to (81.5, 62.4)
- moved R23 17.4 mm to (92.7, 60.3), turned to 180 degrees
- moved R20 17.3 mm to (89.0, 62.4), turned to -90 degrees
- moved R17 15.9 mm to (84.4, 69.3), turned to 180 degrees
- moved TP1 6.39 mm to (91.5, 80.4)
- moved R12 5.32 mm to (69.4, 75.5)
- moved R7 5.32 mm to (69.4, 76.9)
- moved R13 5.32 mm to (71.8, 75.5)
- moved R14 5.32 mm to (69.4, 74.2)
- moved R8 5.32 mm to (71.8, 76.9)
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- renumbered C1 to C3, J1 to J3, R2 to R1, R8 to R12, R9 to R13, R6 to R14, R7 to R15, R1 to R2, R16 to R35, R5 to R6, R10 to R7, R11 to R8, R4 to R9
Connections:
- net Net-(J1-GPIO1_EC) renamed /GPIO1
- J3 pad PA4: 3V3_ALW -> 3V3_CTRL
- J3 pad PA5: unconnected-(J1-3V3_ALW-PadPA5) -> 3V3_ID
- J3 pad PB4: 3V3_ALW -> 3V3_CTRL
- J3 pad PB5: unconnected-(J1-3V3_ALW-PadPB5) -> 3V3_ID
- J3 pad PG1: Net-(J1-GPIO0_EC) -> /GPIO0
- J3 pad PG2: /SSD2_CLKREQ -> /CLKREQ2
- J3 pad PJ3: unconnected-(J1-USB+-PadPJ3) -> /USB+
- J3 pad PK3: unconnected-(J1-USB--PadPK3) -> /USB-
- J3 pad PK7: unconnected-(J1-5V_ALW-PadPK7) -> 5V_ALW
- J3 pad PK8: unconnected-(J1-5V_ALW-PadPK8) -> 5V_ALW
- J3 pad PL1: unconnected-(J1-PWR_GOOD-PadPL1) -> /PWR_GOOD
- J3 pad PL7: unconnected-(J1-5V_ALW-PadPL7) -> 5V_ALW
- J3 pad PL8: unconnected-(J1-5V_ALW-PadPL8) -> 5V_ALW
- J3 pad SA4: /CLKREQ -> /CLKREQ1
- J3 pad SA5: Net-(J1-PEX_RST#) -> /PEX_RST
- J3 pad SC2: /REFCLKA- -> /REFCLKA+
- J3 pad SD2: /REFCLKA+ -> /REFCLKA-
- J3 pad SJ7: unconnected-(J1-DP_A_AUXN-PadSJ7) -> /REFCLKB-
- J3 pad SK7: unconnected-(J1-DP_A_AUXP-PadSK7) -> /REFCLKB+
- R17 pad 1: Net-(U1-SCL) -> GND
- R17 pad 2: /I2C_SCL -> Net-(R17-Pad2)
- R18 pad 1: Net-(U1-SDA) -> 3V3_CTRL
- R18 pad 2: /I2C_SDA -> /CLKREQ1
- R19 pad 1: /CPRSNTA -> /CLK_AUTO_EN1
- R19 pad 2: 3V3_ALW -> /CLKREQ1
- R20 pad 1: /EEPROM_WP -> 3V3_CTRL
- R20 pad 2: GND -> /CLKREQ2
- R21 pad 1: Net-(R12-Pad1) -> /CLK_AUTO_EN2
- R21 pad 2: /CLKREQ -> /CLKREQ2
- R23 pad 1: Net-(J1-PEX_RST#) -> 3V3_CTRL
- R23 pad 2: /PERSTA -> /3V3_CLK_EN2
- R35 pad 1: 3V3_ALW -> Net-(J6-Shield)
- R35 pad 2: /3V3_EEPROM -> GND
- R5 pad 1: /EEPROM_WP -> 3V3_ID
- R6 pad 1: Net-(U1-SDA) -> Net-(J4-Pin_3)
- R9 pad 2: Net-(U1-SCL) -> Net-(J4-Pin_4)
- TP1 pad 1: Net-(J1-GPIO0_EC) -> /PWR_GOOD
- U1 pad 5: Net-(U1-SDA) -> Net-(J4-Pin_3)
- U1 pad 6: Net-(U1-SCL) -> Net-(J4-Pin_4)
Routing:
- net 12V_FAN: track 116.6 -> 0.00 mm
- net /REFCLKB+: track 0.00 -> 101.2 mm, vias 0 -> 2
- net /REFCLKB-: track 0.00 -> 101.2 mm, vias 0 -> 2
- net /USB-: track 0.00 -> 84.9 mm, vias 0 -> 2
- net /USB+: track 0.00 -> 84.9 mm, vias 0 -> 2
- net /PERSTB: track 0.00 -> 77.1 mm, vias 0 -> 2
- net 3V3_CTRL: track 0.00 -> 74.5 mm
- net /CLKREQ1: track 0.00 -> 55.2 mm, vias 0 -> 2
- net /CPRSNTB: track 0.00 -> 54.0 mm, vias 0 -> 2
- net /PEX_RST: track 0.00 -> 48.0 mm, vias 0 -> 2
- net /CLKREQ2: track 0.00 -> 45.5 mm, vias 0 -> 2
- net 5V_ALW: track 0.00 -> 43.5 mm, vias 0 -> 12
- net /SSD2_RST: track 0.00 -> 40.7 mm, vias 0 -> 2
- net Net-(J6-Shield): track 0.00 -> 35.5 mm
- net Net-(J1-GPIO0_EC): track 27.5 -> 0.00 mm, vias 2 -> 0
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- added copper zone on F.Cu, net 12V_FAN
- added copper zone on B.Cu, net 5V_ALW
- added copper zone on F.Cu, net 5V_ALW
Other:
- board size 118.7 x 72.5 mm -> 119 x 73.9 mm
- board text added: "Framework 16 Laptop FXBeam to OCuLink REV 1.2 ENGINEER SAMPLE"
- board text removed: "Framework 16 Laptop FXBeam to OCuLink Card REV 1.1 ENGINEER SAMPLE"

Commit message: finalize rev1.3
Parts:
- added R36: 0R, Resistor_SMD:R_0402_1005Metric, F.Cu at (81.9, 71.8)
- R24, R25: value 9K1 -> 100K
- R26, R27: value 3K9 -> 47K
- R28, R31: value 0R -> 1K
- R29, R32: value 47K -> 100K
- moved J5 5.00 mm to (57.8, 47.5)
- moved R34 5.00 mm to (47.1, 47.1)
- moved C1 0.13 mm to (140.8, 93.4)
- turned R30 to 90 degrees
- turned R33 to 90 degrees
Connections:
- SW1 pad 6: /PEX_RST -> Net-(SW1B-C)
Routing:
- net /USB+: track 84.9 -> 78.5 mm
- net /USB-: track 84.9 -> 78.5 mm
- net /PERSTB: track 77.1 -> 73.6 mm
- net /REFCLKB-: track 101.2 -> 97.9 mm
- net /REFCLKB+: track 101.2 -> 98.0 mm
- net Net-(SW1B-C): track 0.00 -> 2.23 mm
- net /TX3+: track 84.9 -> 82.9 mm
- net /TX3-: track 84.9 -> 82.9 mm
- net /RX1-: track 85.7 -> 83.9 mm
- net /RX1+: track 85.7 -> 83.9 mm
- net /FAN1_PWM: track 55.2 -> 57.0 mm
- net /FAN1_SPD: track 52.2 -> 54.0 mm
- net /TX2+: track 82.2 -> 80.5 mm
- net /TX2-: track 82.2 -> 80.5 mm
- net /RX0-: track 81.0 -> 79.3 mm
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Other:
- outline, holes or cut-outs redrawn
- board text added: "Framework 16 Laptop FXBeam to OCuLink REV 1.3"
- board text removed: "Framework 16 Laptop FXBeam to OCuLink REV 1.2 ENGINEER SAMPLE"

Commit message: finalize rev1.3 for real now... maybe
Parts:
- removed R35: 0R, Resistor_SMD:R_0402_1005Metric
- removed TP1, TP2, TP3: TestPoint_Small, TestPoint:TestPoint_Pad_D1.0mm
Connections:
- J3 pad PL1: /PWR_GOOD -> unconnected-(J3A-PWR_GOOD-PadPL1)
- J6 pad A11: /REFCLKA- -> /REFCLKA+
- J6 pad A12: /REFCLKA+ -> /REFCLKA-
- J6 pad A32: /REFCLKB+ -> /REFCLKB-
- J6 pad A33: /REFCLKB- -> /REFCLKB+
- J6 pad A35: /RX6- -> /RX6+
- J6 pad A36: /RX6+ -> /RX6-
- J6 pad A38: /RX7- -> /RX7+
- J6 pad A39: /RX7+ -> /RX7-
- J6 pad MP: Net-(J6-Shield) -> GND
Routing:
- net 12V_FAN: track 0.00 -> 92.3 mm, vias 0 -> 4
- net /FAN1_SPD: track 54.0 -> 92.0 mm, vias 2 -> 4
- net Net-(J6-Shield): track 35.5 -> 0.00 mm
- net /FAN1_PWM: track 57.0 -> 89.8 mm, vias 2 -> 4
- net /GPIO0: track 25.6 -> 0.00 mm, vias 2 -> 0
- net /GPIO1: track 23.6 -> 0.00 mm, vias 2 -> 0
- net /PWR_GOOD: track 22.7 -> 0.00 mm, vias 2 -> 0
- net /CPRSNTA: track 108.7 -> 88.9 mm, vias 4 -> 2
- net /PERSTA: track 103.6 -> 98.7 mm, vias 4 -> 2
- net /RX3-: track 74.3 -> 69.4 mm
- net /RX3+: track 74.3 -> 69.6 mm
- net /RX5-: track 73.0 -> 68.6 mm
- net /RX5+: track 73.0 -> 68.6 mm
- net /REFCLKB+: track 98.0 -> 94.6 mm
- net /REFCLKB-: track 97.9 -> 94.7 mm
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- added copper zone on B.Cu, net 12V_FAN
